File: bluepill_yoke.kicad_pcb (KiCad board)
At the start: 2 copper layers, 40 x 53 mm, 71 parts, among them J1 Conn_01x03_Socket, J2 Conn_01x03_Socket, J3 Conn_01x03_Socket, J4 Conn_01x03_Socket, J5 Conn_01x09_Socket, J6 Conn_01x07_Socket, J7 Conn_01x03_Socket, U1 YAAJ_BluePill_Part_Like

Commit message: Finished pcb
Parts:
- removed JP9: SolderJumper_2_Bridged, Jumper:SolderJumper-2_P1.3mm_Open_TrianglePad1.0x1.5mm
- added J8: Conn_01x02, Connector_PinHeader_2.54mm:PinHeader_1x02_P2.54mm_Vertical, F.Cu at (118.3, 65.8)
- added J9: Conn_01x03, Connector_PinHeader_2.54mm:PinHeader_1x03_P2.54mm_Horizontal, F.Cu at (118.4, 62.1)
- added JP23: SolderJumper_2_Open, Jumper:SolderJumper-2_P1.3mm_Open_TrianglePad1.0x1.5mm, B.Cu at (115.4, 81.6)
- JP1, JP10, JP11, JP12, JP13, JP14, JP15, JP16, JP17, JP18, JP19, JP2, JP20, JP21, JP22, JP3, JP4, JP5, JP6, JP7, JP8: value SolderJumper_2_Bridged -> SolderJumper_2_Open
- moved JP19 13.2 mm to (108.8, 81.2), turned to 180 degrees
- moved JP22 4.40 mm to (115.4, 85.9)
- moved JP21 3.50 mm to (115.2, 89.5)
- moved JP20 3.30 mm to (115.2, 92.8)
- moved JP17 3.22 mm to (108.8, 87.6)
- moved JP18 3.22 mm to (108.8, 84.6)
- moved R22 1.31 mm to (105.2, 81.2)
- moved J7 1.00 mm to (91.5, 71.0)
- moved R21 0.88 mm to (105.4, 84.8)
- moved R20 0.88 mm to (105.4, 87.2)
- moved C22 0.81 mm to (108.8, 81.2)
- moved J4 0.70 mm to (118.3, 77.8)
- moved C4 0.41 mm to (121.9, 80.6)
- moved C10 0.36 mm to (90.4, 87.8)
- moved C12 0.33 mm to (90.5, 93.0)
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Connections:
- JP17 pad 1: /PA3 -> /PA5
- JP17 pad 2: /S13_BLU -> /S12_YEL
- JP18 pad 1: /PA4 -> /PA6
- JP18 pad 2: /S14_GRY -> /S13_BLU
- JP19 pad 1: /PA0 -> /PA7
- JP19 pad 2: Net-(J1-Pin_2) -> /S14_GRY
- JP20 pad 1: /PA1 -> /PA0
- JP20 pad 2: Net-(J2-Pin_2) -> Net-(J1-Pin_2)
- JP21 pad 1: /PA2 -> /PA1
- JP21 pad 2: Net-(J3-Pin_2) -> Net-(J2-Pin_2)
- JP22 pad 1: /PA3 -> /PA2
- JP22 pad 2: Net-(J4-Pin_2) -> Net-(J3-Pin_2)
Routing:
- net /PA5: track 0.00 -> 9.60 mm
- net /PA6: track 0.00 -> 9.41 mm
- net /PA7: track 0.00 -> 8.33 mm
- net Net-(J8-Pin_2): track 0.00 -> 3.75 mm
- net Net-(J8-Pin_1): track 0.00 -> 3.75 mm
- net /PA4: track 2.25 -> 0.00 mm
- net /PA2: track 4.75 -> 2.53 mm
- net /PA3: track 6.67 -> 4.48 mm
- net Net-(J4-Pin_2): track 8.74 -> 9.56 mm
- net /S12_YEL: track 34.4 -> 35.1 mm
- net /S13_BLU: track 26.2 -> 25.7 mm
- net GND: vias 39 -> 44
Other:
- outline, holes or cut-outs redrawn
- board text added: "3V3 PA0 GND"
- board text added: "3V3 PA1 GND"
- board text added: "3V3 PA2 GND"
- board text added: "3V3 PA3 GND"
- board text added: "BLU GRY WHT PPL ORG GRN YEL"
- board text added: "DIO CLK GND"
- board text added: "ORG PPL WHT GRY BLK BLU BRN YEL GND"
- board text added: "YEL BLU GRY"
