File: bluepill_yoke.kicad_sch (KiCad schematic)
At the start: 71 parts, among them J1 Conn_01x03_Socket, J2 Conn_01x03_Socket, J3 Conn_01x03_Socket, J4 Conn_01x03_Socket, J5 Conn_01x09_Socket, J6 Conn_01x07_Socket, J7 Conn_01x03_Socket, U1 YAAJ_BluePill_Part_Like

Commit message: Finished pcb
Parts:
- removed JP1, JP10, JP11, JP12, JP13, JP14, JP15, JP16, JP17, JP18, JP19, JP2, JP20, JP21, JP22, JP3, JP4, JP5, JP6, JP7, JP8, JP9: SolderJumper_2_Bridged, Jumper:SolderJumper-2_P1.3mm_Open_TrianglePad1.0x1.5mm, symbol Jumper:SolderJumper_2_Bridged
- added J8: Conn_01x02, Connector_PinHeader_2.54mm:PinHeader_1x02_P2.54mm_Vertical, symbol Connector_Generic:Conn_01x02
- added J9: Conn_01x03, Connector_PinHeader_2.54mm:PinHeader_1x03_P2.54mm_Horizontal, symbol Connector_Generic:Conn_01x03
- added JP1, JP10, JP11, JP12, JP13, JP14, JP15, JP16, JP17, JP18, JP19, JP2, JP20, JP21, JP22, JP23, JP3, JP4, JP5, JP6, JP7, JP8: SolderJumper_2_Open, Jumper:SolderJumper-2_P1.3mm_Open_TrianglePad1.0x1.5mm, symbol Jumper:SolderJumper_2_Open
Connections:
- net GND: now also J9.3 (Pin_3)
- net PA0: now also JP20.1 (A)
- net PA1: now also JP21.1 (A)
- net PA2: now also JP22.1 (A)
- net PA3: now also JP23.1 (A)
- net PA5: now also JP17.1 (A)
- net PA6: now also JP18.1 (A)
- net PA7: now also JP19.1 (A)
- net PB0: now also JP1.1 (A)
- net PB1: now also JP2.1 (A)
- net PB10: now also JP11.1 (A)
- net PB11: now also JP12.1 (A)
- net PB12: now also JP13.1 (A)
- net PB13: now also JP14.1 (A)
- net PB14: now also JP15.1 (A)
- net PB15: now also JP16.1 (A)
- net PB3: now also JP3.1 (A)
- net PB4: now also JP4.1 (A)
- net PB5: now also JP5.1 (A)
- net PB6: now also JP6.1 (A)
- net PB7: now also JP7.1 (A)
- net PB8: now also JP8.1 (A)
- net PB9: now also JP10.1 (A)
- net S10_BRN: now also JP7.2 (B)
- net S11_YEL: now also JP8.2 (B)
- net S12_YEL: now also JP17.2 (B)
- net S13_BLU: now also JP18.2 (B)
- net S14_GRY: now also JP19.2 (B)
- net S15_PPL: now also JP13.2 (B)
- net S16_ORG: now also JP14.2 (B)
- net S17_GRN: now also JP15.2 (B)
- net S18_YEL: now also JP16.2 (B)
- net S1_BLU: now also JP10.2 (B)
- net S2_ORG: now also JP1.2 (B)
- net S3_GRY: now also JP11.2 (B)
- net S4_WHT: now also JP12.2 (B)
- net S5_PPL: now also JP2.2 (B)
- net S6_WHT: now also JP3.2 (B)
- net S7_GRY: now also JP4.2 (B)
- net S8_BLK: now also JP5.2 (B)
- net S9_BLU: now also JP6.2 (B)
- net at C2.1, J2.2 (Pin_2): now also JP21.2 (B)
- net at C1.1, J1.2 (Pin_2): now also JP20.2 (B)
- net at C4.1, J4.2 (Pin_2): now also JP23.2 (B)
- net at C3.1, J3.2 (Pin_2): now also JP22.2 (B)
- new net: J8.1 (Pin_1), J9.1 (Pin_1)
- new net: J8.2 (Pin_2), J9.2 (Pin_2)
Other:
- moved on the sheet: C13, C14, C15, C16, C17, C18, C19, C20, C21, C22, J6, J7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
